Commit message: "mujoco simulator update"

File: models/test_2/test_2.urdf (robot description, URDF)
Before this commit: robot test_2, 7 links, 6 joints
Joints:
- joint joint_3: axis 1.000000 0.000000 0.000000 -> -1.000000 -0.000000 0.000000
- joint joint_4: axis 1.000000 0.000000 0.000000 -> -1.000000 -0.000000 0.000000
- joint joint_5: axis 1.000000 0.000000 0.000000 -> -1.000000 -0.000000 0.000000
