Commit message: new friction synergy framework

File: tests/simple_fold.urdf (robot description, URDF)
Before this commit: robot simple_fold, 2 links, 1 joints
Links:
- link face_0: geometry visual mesh filename=meshes/face_0.stl scale=1.0 1.0 1.0
- link face_1: geometry visual mesh filename=meshes/face_1.stl scale=1.0 1.0 1.0
Joints:
- joint joint_0: axis 0.0 1.0 0.0 -> -0.000000 -1.000000 0.000000; origin xyz=2.5 1.5 0.001 rpy=0 0 0 -> xyz=2.500000 1.500000 0.000000 rpy=0 0 0
