Commit message: doc updates

File: models/ohd_7/ohd_7.urdf (robot description, URDF)
Before this commit: robot ohd_7, 16 links, 15 joints
Links:
- link face_0: geometry collision mesh filename=meshes/face_0.stl scale=1.0 1.0 1.0; visual mesh filename=meshes/face_0.stl scale=1.0 1.0 1.0
- link face_1: geometry collision mesh filename=meshes/face_1.stl scale=1.0 1.0 1.0; visual mesh filename=meshes/face_1.stl scale=1.0 1.0 1.0
- link face_10: geometry collision mesh filename=meshes/face_10.stl scale=1.0 1.0 1.0; visual mesh filename=meshes/face_10.stl scale=1.0 1.0 1.0
- link face_11: geometry collision mesh filename=meshes/face_11.stl scale=1.0 1.0 1.0; visual mesh filename=meshes/face_11.stl scale=1.0 1.0 1.0
- link face_12: geometry collision mesh filename=meshes/face_12.stl scale=1.0 1.0 1.0; visual mesh filename=meshes/face_12.stl scale=1.0 1.0 1.0
- link face_13: geometry collision mesh filename=meshes/face_13.stl scale=1.0 1.0 1.0; visual mesh filename=meshes/face_13.stl scale=1.0 1.0 1.0
- link face_14: geometry collision mesh filename=meshes/face_14.stl scale=1.0 1.0 1.0; visual mesh filename=meshes/face_14.stl scale=1.0 1.0 1.0
- link face_15: geometry collision mesh filename=meshes/face_15.stl scale=1.0 1.0 1.0; visual mesh filename=meshes/face_15.stl scale=1.0 1.0 1.0
- link face_2: geometry collision mesh filename=meshes/face_2.stl scale=1.0 1.0 1.0; visual mesh filename=meshes/face_2.stl scale=1.0 1.0 1.0
- link face_3: geometry collision mesh filename=meshes/face_3.stl scale=1.0 1.0 1.0; visual mesh filename=meshes/face_3.stl scale=1.0 1.0 1.0
- link face_4: geometry collision mesh filename=meshes/face_4.stl scale=1.0 1.0 1.0; visual mesh filename=meshes/face_4.stl scale=1.0 1.0 1.0
- link face_5: geometry collision mesh filename=meshes/face_5.stl scale=1.0 1.0 1.0; visual mesh filename=meshes/face_5.stl scale=1.0 1.0 1.0
- link face_6: geometry collision mesh filename=meshes/face_6.stl scale=1.0 1.0 1.0; visual mesh filename=meshes/face_6.stl scale=1.0 1.0 1.0
- link face_7: geometry collision mesh filename=meshes/face_7.stl scale=1.0 1.0 1.0; visual mesh filename=meshes/face_7.stl scale=1.0 1.0 1.0
- link face_8: geometry collision mesh filename=meshes/face_8.stl scale=1.0 1.0 1.0; visual mesh filename=meshes/face_8.stl scale=1.0 1.0 1.0
- link face_9: geometry collision mesh filename=meshes/face_9.stl scale=1.0 1.0 1.0; visual mesh filename=meshes/face_9.stl scale=1.0 1.0 1.0
